Commit message: final test for tw initial global maps

File: src/mir_robot/mir_description/urdf/include/mir_v1.urdf.xacro (robot description, xacro)
@@ -269,5 +269,5 @@
     <xacro:set_all_wheel_frictions prefix="${prefix}"/>
     <xacro:p3d_base_controller prefix="${prefix}" />
-    <!-- 3d_camera-->
+    <!-- Add the kinect_camera model to the robot model and add the camera plugin-->
     <xacro:sensor_kinect parent="${prefix}base_link" cam_px="0.2" cam_py="0.0" cam_pz="1.0" cam_or="0" cam_op="0.08" cam_oy="0" />
     <xacro:sim_3dsensor_kinect />

File: src/openni_camera/openni_description/model/kinect.urdf.xacro (robot description, xacro)
@@ -20,5 +20,5 @@
       <child link="camera_link"/>
     </joint>
-      <link name="camera_link">
+    <link name="camera_link">
       <visual>
        <origin xyz="0 0 0" rpy="0 0 ${pi/2}"/>
@@ -44,17 +44,17 @@
          files. However, for Gazebo simulation we need them, so we add them here.
          (Hence, don't publish them additionally!) -->
-	<joint name="camera_depth_joint" type="fixed">
-	  <origin xyz="0 ${2 * -cam_py} 0" rpy="0 0 0" />
-	  <parent link="camera_rgb_frame" />
-	  <child link="camera_depth_frame" />
-	</joint>
-	<link name="camera_depth_frame"/>
-	<joint name="camera_depth_optical_joint" type="fixed">
-	  <origin xyz="0 0 0" rpy="${-pi/2} 0 ${-pi/2}" />
-	  <parent link="camera_depth_frame" />
-	  <child link="camera_depth_optical_frame" />
-	</joint>
-	<link name="camera_depth_optical_frame"/>
-	<!-- Kinect sensor for simulation -->
+    <joint name="camera_depth_joint" type="fixed">
+      <origin xyz="0 ${2 * -cam_py} 0" rpy="0 0 0" />
+      <parent link="camera_rgb_frame" />
+      <child link="camera_depth_frame" />
+    </joint>
+    <link name="camera_depth_frame"/>
+    <joint name="camera_depth_optical_joint" type="fixed">
+      <origin xyz="0 0 0" rpy="${-pi/2} 0 ${-pi/2}" />
+      <parent link="camera_depth_frame" />
+      <child link="camera_depth_optical_frame" />
+    </joint>
+    <link name="camera_depth_optical_frame"/>
+    <!-- Kinect sensor for simulation -->
 	<sim_3dsensor_kinect/>
   </xacro:macro>

File: src/openni_camera/openni_description/model/kinect_gazebo.urdf.xacro (robot description, xacro)
@@ -8,5 +8,5 @@
         <update_rate>30.0</update_rate>
         <camera>
-          <horizontal_fov>1.012</horizontal_fov>
+          <horizontal_fov>1.047198</horizontal_fov>
           <image>
             <format>B8G8R8</format>
@@ -15,5 +15,5 @@
           </image>
           <clip>
-            <near>0.1</near>
+            <near>0.5</near>
             <far>3.5</far>
           </clip>
@@ -35,6 +35,6 @@
           <distortion_t1>0.0</distortion_t1>
           <distortion_t2>0.0</distortion_t2>
-          <!--<pointCloudCutoff>0.4</pointCloudCutoff>-->
-          <!--<pointCloudCutoffMax>3.0</pointCloudCutoffMax>-->
+          <pointCloudCutoff>0.5</pointCloudCutoff>
+          <pointCloudCutoffMax>3.5</pointCloudCutoffMax>
         </plugin>
       </sensor>
